File: Flight Computer PCB/Flight Computer PCB.kicad_pcb (KiCad board)
At the start: 4 copper layers, 45 x 40 mm, 58 parts, among them IC1 STM32F745VGT6, J1 TYPE-C_16PIN_2MD__073_, J3 SM12B-GHS-TB, J4 Conn_01x05_Pin, U2 MPU-6000, U3 USBLC6-2SC6, U4 BMP280, U5 W25Q128JVSIQ, U6 MCP1700T-3302E/TT, Y1 8MHz

Commit message: Finished pcb
Parts:
- added R19: 50, Resistor_SMD:R_0805_2012Metric, F.Cu at (236.7, 77.0)
- added R20: 50, Resistor_SMD:R_0805_2012Metric, F.Cu at (227.1, 77.0)
- added R21: 50, Resistor_SMD:R_0805_2012Metric, F.Cu at (230.3, 77.0)
- added R22: 50, Resistor_SMD:R_0805_2012Metric, F.Cu at (220.7, 77.0)
- added R23: 50, Resistor_SMD:R_0805_2012Metric, F.Cu at (223.9, 77.0)
- added R24: 50, Resistor_SMD:R_0805_2012Metric, F.Cu at (214.3, 77.0)
- added R25: 50, Resistor_SMD:R_0805_2012Metric, F.Cu at (217.4, 77.0)
- added R7: 50, Resistor_SMD:R_0805_2012Metric, F.Cu at (233.5, 77.0)
- moved J4 14.0 mm to (247.1, 77.1), turned to 0 degrees
Routing:
- net /RESET: track 40.4 -> 99.5 mm
- net /RC_RX: track 0.00 -> 34.5 mm, vias 0 -> 2
- net /RC_TX: track 0.00 -> 33.4 mm, vias 0 -> 2
- net /VTX_TX: track 0.00 -> 28.1 mm, vias 0 -> 2
- net /VTX_RX: track 0.00 -> 27.0 mm, vias 0 -> 2
- net /USB_TX: track 0.00 -> 23.3 mm, vias 0 -> 4
- net /USB_RX: track 0.00 -> 23.1 mm, vias 0 -> 2
- net /GPS_RX: track 0.00 -> 20.8 mm
- net /GPS_TX: track 0.00 -> 18.7 mm
- net /SWDCLK: track 9.45 -> 20.9 mm
- net +3.3V: track 56.3 -> 63.8 mm, vias 17 -> 21
- net GND: track 115.2 -> 122.2 mm, vias 38 -> 45
- net /USB_TX_PAD: track 0.00 -> 6.34 mm
- net /RC_RX_PAD: track 0.00 -> 6.34 mm
- net /VTX_TX_PAD: track 0.00 -> 6.34 mm
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- added copper zone on B.Cu, net GND
- added copper zone on F.Cu, net GND
Other:
- board size 45 x 40 mm -> 50 x 50 mm
