File: Flight Computer PCB/Flight Computer PCB.kicad_sch (KiCad schematic)
At the start: 35 parts, among them IC1 STM32F745VGT6, J1 TYPE-C_16PIN_2MD__073_, SW1 SW_SPDT, U2 MPU-6000, U3 USBLC6-2SC6, U4 BMP280, U5 W25Q128JVSIQ, Y1 24MHz

Commit message: Initial commit
Parts:
- added C21, C22: 1u, symbol Device:C
- added C23: 10u, symbol Device:C
- added D1: D_TVS, symbol Device:D_TVS
- added J2: Conn_01x06_Pin, Connector_PinHeader_2.54mm:PinHeader_1x06_P2.54mm_Vertical, symbol Connector:Conn_01x06_Pin
- added J3: Conn_01x08_Pin, symbol Connector:Conn_01x08_Pin
- added R7, R8, R9: 50, symbol Device:R
- added U6: MCP1700T-3302E/TT, Package_TO_SOT_SMD:SOT-89-3, symbol Regulator_Linear:MCP1700x-330xxMB
- C1, C11, C12, C13, C14, C15, C16, C17, C18, C2, C20, C3, C4, C5, C6, C7, C8, R1, R2, R3, R4: footprint Capacitor_SMD:C_0402_1005Metric -> (none)
- C10, C9: value 18pF -> ~; footprint Capacitor_SMD:C_0402_1005Metric -> (none)
- IC1: footprint QFP50P1600X1600X160-100N -> 02Footprints:QFP50P1600X1600X160-100N
- Y1: value 24MHz -> 8MHz; footprint Crystal:Crystal_SMD_3225-4Pin_3.2x2.5mm -> (none)
Connections:
- net HES_OUT is gone; now on net HSE_OUT: C10.1, Y1.3
- net +3.3V: now also C21.1, J2.1 (Pin_1), U6.3 (VO)
- net ESC_RX: now also R8.1
- net ESC_TX: now also R9.1
- net GND: now also C21.2, C22.2, C23.2, D1.1 (A1), J2.3 (Pin_3), J3.4 (Pin_4), U6.1 (GND)
- net RESET: now also J2.5 (Pin_5)
- net SWDCLK: now also J2.4 (Pin_4)
- net SWDIO: now also J2.2 (Pin_2)
- net SWO: now also J2.6 (Pin_6), R7.1; no longer IC1.89 (PB3-SYS_JTDO-SWO)
- net TIM1_C1: now also J3.8 (Pin_8)
- net TIM1_C2: now also J3.7 (Pin_7)
- net TIM1_C3: now also J3.6 (Pin_6)
- net TIM1_C4: now also J3.5 (Pin_5)
- net VBUS: now also D1.2 (A2)
- net 5V_OUT renamed +5V
- net +5V: now also C22.1, C23.1, J3.1 (Pin_1), U6.2 (VI)
- new net: J3.3 (Pin_3), R9.2
- new net: J3.2 (Pin_2), R8.2
- new net SWO_R: IC1.89 (PB3-SYS_JTDO-SWO), R7.2
- no-connect marks 8 -> 66
Other:
- moved on the sheet: C1, C10, C11, C14, C16, C17, C2, C3, C4, C9, IC1, J1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

Commit message: Schematic update
Parts:
- removed J3: Conn_01x08_Pin, symbol Connector:Conn_01x08_Pin
- removed SW1: SW_SPDT, 02Footprints:SW-SMD_SSSS810701, symbol Switch:SW_SPDT
- added D2, D3: D, symbol Device:D
- added F1: 300mA, symbol Device:Polyfuse
- added J4: Conn_01x12_Pin, symbol Connector:Conn_01x12_Pin
- added R10, R11, R12, R13: 50, symbol Device:R
- added R14, R15: 5k1, symbol Device:R
Connections:
- net BOOT_R is gone; now on net GND: R3.2
- net +3.3V: now also R14.1, R15.1
- net +5V: now also D2.1 (K), D3.1 (K), F1.1; no longer C22.1, U3.2 (GND), U6.2 (VI)
- net ESC_RX: now also R8.2, J4.3 (Pin_3)
- net ESC_TX: now also R9.2, J4.4 (Pin_4)
- net GND: now also U3.2 (GND), J4.11 (Pin_11), J4.2 (Pin_2), J4.5 (Pin_5), J4.7 (Pin_7), J4.9 (Pin_9)
- net I2C1_SCL: now also R14.2
- net I2C1_SDA: now also R15.2
- net TIM1_C1: now also R12.1
- net TIM1_C2: now also R13.1
- net TIM1_C3: now also R11.1
- net TIM1_C4: now also R10.1
- net VBUS: now also D2.2 (A)
- new net: C22.1, F1.2, U6.2 (VI)
- new net ESC_5V: D3.2 (A), J4.1 (Pin_1)
- new net ESC_CH1: J4.12 (Pin_12), R12.2
- new net ESC_CH2: J4.10 (Pin_10), R13.2
- new net ESC_CH3: J4.8 (Pin_8), R11.2
- new net ESC_CH4: J4.6 (Pin_6), R10.2
Other:
- moved on the sheet: C1, C14, C15, C18, C19, C2, C20, C21, C22, C23, C3, C4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

Commit message: Schematic update
Parts:
- removed D2, D3: D, symbol Device:D
- added D2, D4: D_Schottky, symbol Device:D_Schottky
- C10, C9: value ~ -> 12p
- F1: value 300mA -> 250mA
- Y1: footprint (none) -> Crystal:Crystal_SMD_3225-4Pin_3.2x2.5mm
Connections:
- net +5V: now also D2.1 (K), D4.1 (K)
- net ESC_5V: now also D2.2 (A)
- net VBUS: now also D4.2 (A)
Changed lines of the file:
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@@
 	)
 	(symbol
-		(lib_id "Device:D")
-		(at 368.3 208.28 0)
-		(unit 1)
-		(exclude_from_sim no)
-		(in_bom yes)
-		(on_board yes)
-		(dnp no)
-		(fields_autoplaced yes)
-		(property "Reference" "D3"
-			(at 368.3 201.93 0)
-			(effects
-				(font
-					(size 1.27 1.27)
-				)
-			)
-		)
-		(property "Value" "D"
-			(at 368.3 204.47 0)
-			(effects
-				(font
-					(size 1.27 1.27)
-				)
-			)
-		)
-		(property "Footprint" ""
-			(at 368.3 208.28 0)
-			(effects
-				(font
-					(size 1.27 1.27)
-				)
-				(hide yes)
-			)
-		)
-		(property "Datasheet" "~"
-			(at 368.3 208.28 0)
-			(effects
-				(font
-					(size 1.27 1.27)
-				)
-				(hide yes)
-			)
-		)
-		(property "Description" "Diode"
-			(at 368.3 208.28 0)
-			(effects
-				(font
-					(size 1.27 1.27)
-				)
-				(hide yes)
-			)
-		)
-		(property "Sim.Device" "D"
-			(at 368.3 208.28 0)
-			(effects
-				(font
-					(size 1.27 1.27)
-				)
-				(hide yes)
-			)
-		)
-		(property "Sim.Pins" "1=K 2=A"
-			(at 368.3 208.28 0)
-			(effects
-				(font
-					(size 1.27 1.27)
-				)
-				(hide yes)
-			)
-		)
-		(pin "2"
-		)
-		(pin "1"
-		)
-		(instances
-			(project "Flight Computer PCB"
-				(path "/71f2845f-655b-4c65-8656-911ca469396e"
-					(reference "D3")
-					(unit 1)
-				)
-			)
-		)
-	)
-	(symbol
-		(lib_id "Device:D")
-		(at 127 231.14 0)
-		(unit 1)
-		(exclude_from_sim no)
-		(in_bom yes)
-		(on_board yes)
-		(dnp no)
-		(fields_autoplaced yes)
-		(property "Reference" "D2"
-			(at 127 224.79 0)
-			(effects
-				(font
-					(size 1.27 1.27)
-				)
-			)
-		)
-		(property "Value" "D"
-			(at 127 227.33 0)
-			(effects
-				(font
-					(size 1.27 1.27)
-				)
-			)
-		)
-		(property "Footprint" ""
-			(at 127 231.14 0)
-			(effects
-				(font
-					(size 1.27 1.27)
-				)
-				(hide yes)
-			)
-		)
-		(property "Datasheet" "~"
-			(at 127 231.14 0)
-			(effects
-				(font
-					(size 1.27 1.27)
-				)
-				(hide yes)
-			)
-		)
-		(property "Description" "Diode"
-			(at 127 231.14 0)
-			(effects
-				(font
-					(size 1.27 1.27)
-				)
-				(hide yes)
-			)
-		)
-		(property "Sim.Device" "D"
-			(at 127 231.14 0)
-			(effects
-				(font
-					(size 1.27 1.27)
-				)
-				(hide yes)
-			)
-		)
-		(property "Sim.Pins" "1=K 2=A"
-			(at 127 231.14 0)
-			(effects
-				(font
-					(size 1.27 1.27)
-				)
-				(hide yes)
-			)
-		)
-		(pin "2"
-		)
-		(pin "1"
-		)
-		(instances
-			(project ""
-				(path "/71f2845f-655b-4c65-8656-911ca469396e"
-					(reference "D2")
-					(unit 1)
-				)
-			)
-		)
-	)
-	(symbol
 		(lib_id "Device:R")
 		(at 365.76 215.9 90)
@@
 			)
 		)
-		(property "Value" "~"
+		(property "Value" "12p"
 			(at 54.61 91.4399 0)
 			(effects
@@
 			)
 		)
-		(property "Value" "~"
+		(property "Value" "12p"
 			(at 39.37 91.4399 0)
 			(effects
@@
 			)
 		)
-		(property "Footprint" ""
+		(property "Footprint" "Crystal:Crystal_SMD_3225-4Pin_3.2x2.5mm"
 			(at 48.26 83.82 0)
 			(effects
@@
 	)
 	(symbol
+		(lib_id "Device:D_Schottky")
+		(at 127 231.14 0)
+		(unit 1)
+		(exclude_from_sim no)
+		(in_bom yes)
+		(on_board yes)
+		(dnp no)
+		(fields_autoplaced yes)
+		(property "Reference" "D4"
+			(at 126.6825 224.79 0)
+			(effects
+				(font
+					(size 1.27 1.27)
+				)
+			)
+		)
+		(property "Value" "D_Schottky"
+			(at 126.6825 227.33 0)
+			(effects
+				(font
+					(size 1.27 1.27)
+				)
+			)
+		)
+		(property "Footprint" ""
+			(at 127 231.14 0)
+			(effects
+				(font
+					(size 1.27 1.27)
+				)
+				(hide yes)
+			)
+		)
+		(property "Datasheet" "~"
+			(at 127 231.14 0)
+			(effects
+				(font
+					(size 1.27 1.27)
+				)
+				(hide yes)
+			)
+		)
+		(property "Description" "Schottky diode"
+			(at 127 231.14 0)
+			(effects
+				(font
+					(size 1.27 1.27)
+				)
+				(hide yes)
+			)
+		)
+		(pin "1"
+		)
+		(pin "2"
+		)
+		(instances
+			(project ""
+				(path "/71f2845f-655b-4c65-8656-911ca469396e"
+					(reference "D4")
+					(unit 1)
+				)
+			)
+		)
+	)
+	(symbol
 		(lib_id "Device:R")
 		(at 36.83 54.61 90)
@@
 	)
 	(symbol
+		(lib_id "Device:D_Schottky")
+		(at 368.3 208.28 0)
+		(unit 1)
+		(exclude_from_sim no)
+		(in_bom yes)
+		(on_board yes)
+		(dnp no)
+		(fields_autoplaced yes)
+		(property "Reference" "D2"
+			(at 367.9825 201.93 0)
+			(effects
+				(font
+					(size 1.27 1.27)
+				)
+			)
+		)
+		(property "Value" "D_Schottky"
+			(at 367.9825 204.47 0)
+			(effects
+				(font
+					(size 1.27 1.27)
+				)
+			)
+		)
+		(property "Footprint" ""
+			(at 368.3 208.28 0)
+			(effects
+				(font
+					(size 1.27 1.27)
+				)
+				(hide yes)
+			)
+		)
+		(property "Datasheet" "~"
+			(at 368.3 208.28 0)
+			(effects
+				(font
+					(size 1.27 1.27)
+				)
+				(hide yes)
+			)
+		)
+		(property "Description" "Schottky diode"
+			(at 368.3 208.28 0)
+			(effects
+				(font
+					(size 1.27 1.27)
+				)
+				(hide yes)
+			)
+		)
+		(pin "1"
+		)
+		(pin "2"
+		)
+		(instances
+			(project "Flight Computer PCB"
+				(path "/71f2845f-655b-4c65-8656-911ca469396e"
+					(reference "D2")
+					(unit 1)
+				)
+			)
+		)
+	)
+	(symbol
 		(lib_id "Device:C")
 		(at 167.64 167.64 0)
@@
 		)
 		(property "Value" "Conn_01x12_Pin"
-			(at 390.525 205.74 0)
+			(at 390.398 204.978 0)
 			(effects
 				(font
@@
 			)
 		)
-		(property "Value" "300mA"
+		(property "Value" "250mA"
 			(at 31.75 195.5799 0)
 			(effects

Commit message: Finished schematic
Parts:
- removed J2: Conn_01x06_Pin, Connector_PinHeader_2.54mm:PinHeader_1x06_P2.54mm_Vertical, symbol Connector:Conn_01x06_Pin
- removed J4: Conn_01x12_Pin, symbol Connector:Conn_01x12_Pin
- removed R7: 50, symbol Device:R
- added D3, D5, D6: LED, LED_SMD:LED_0805_2012Metric, symbol Device:LED
- added J3: SM12B-GHS-TB, 02Footprints:CONN_SM12B-GHS-TB_JST, symbol SM12B-GHS-TB(LF)(SN):SM12B-GHS-TB
- added J4: Conn_01x05_Pin, Connector_PinHeader_2.54mm:PinHeader_1x05_P2.54mm_Horizontal, symbol Connector:Conn_01x05_Pin
- added R16, R17, R18: 330, Resistor_SMD:R_0805_2012Metric, symbol Device:R
- C1, C10, C11, C12, C13, C14, C15, C16, C17, C18, C19, C2, C20, C21, C22, C23, C3, C4, C5, C6, C7, C8, C9, D1, D2, D4, F1: footprint (none) -> Capacitor_SMD:C_0805_2012Metric
- IC1: footprint 02Footprints:QFP50P1600X1600X160-100N -> QFP50P1600X1600X160-100N
- R1, R10, R11, R12, R13, R14, R15, R2, R3, R4, R5, R6, R8, R9: footprint (none) -> Resistor_SMD:R_0805_2012Metric
- U6: footprint Package_TO_SOT_SMD:SOT-89-3 -> Package_TO_SOT_SMD:SOT-23
Connections:
- net LED/Buzzer is gone; now on net IMU_MISO: IC1.90 (PB4-IMU_MISO)
- net SWO_R is gone; now on net IMU_SCK: IC1.89 (PB3-IMU_SCK)
- net +3.3V: now also J4.5 (Pin_5), R18.2
- net ESC_5V: now also J3.12, R16.2
- net ESC_CH1: now also J3.1
- net ESC_CH2: now also J3.3
- net ESC_CH3: now also J3.5
- net ESC_CH4: now also J3.7
- net ESC_RX: now also R9.1; no longer R8.1, R8.2
- net ESC_TX: now also R8.1; no longer R9.1, R9.2
- net GND: now also D3.1 (K), D5.1 (K), D6.1 (K), J3.11, J3.2, J3.4, J3.6, J3.8, J4.3 (Pin_3)
- net I2C1_SCL: now also IC1.95 (PB8-I2C1_SCL); no longer IC1.92 (PB6-I2C1_SCL)
- net I2C1_SDA: now also IC1.96 (PB9-I2C1_SDA); no longer IC1.93 (PB7-I2C1_SDA)
- net IMU_CS: now also IC1.92 (PB6-IMU_INT); no longer IC1.32 (PC4)
- net IMU_INT: now also IC1.93 (PB7-IMU_CS); no longer IC1.28 (PA4)
- net IMU_MISO: no longer IC1.30 (PA6-IMU_MISO)
- net IMU_MOSI: now also IC1.91 (PB5-IMU_MOSI); no longer IC1.31 (PA7-SPI_MOSI)
- net IMU_SCK: no longer IC1.29 (PA5-IMU_SCK)
- net RESET: now also J4.1 (Pin_1)
- net SWDCLK: now also J4.2 (Pin_2)
- net SWDIO: now also J4.4 (Pin_4)
- net VBUS: now also R17.2
- net 5V_LDO_IN: now reaches C22.1, F1.2, U6.2 (VI)
- net IMU_3V3: now reaches C4.1, R6.2, U2.13 (VDD)
- new net: D3.2 (A), R16.1
- new net: D5.2 (A), R17.1
- new net: D6.2 (A), R18.1
- new net ESC_RX-C: J3.9, R9.2
- new net ESC_TX-C: J3.10, R8.2
Other:
- moved on the sheet: F1, IC1

Commit message: Finished pcb
Parts:
- added R19, R20, R21, R22, R23, R24, R25, R7: 50, Resistor_SMD:R_0805_2012Metric, symbol Device:R
- IC1: footprint QFP50P1600X1600X160-100N -> 02Footprints:QFP50P1600X1600X160-100N
Connections:
- net GPS_RX: now also R22.1
- net GPS_TX: now also R23.1
- net RC_RX: now also R24.1
- net RC_TX: now also R25.1
- net USB_RX: now also R20.1
- net USB_TX: now also R21.1
- net VTX_RX: now also R7.1
- net VTX_TX: now also R19.1
- new net GPS_RX_PAD: R22.2
- new net GPS_TX_PAD: R23.2
- new net RC_RX_PAD: R24.2
- new net RC_TX_PAD: R25.2
- new net USB_RX_PAD: R20.2
- new net USB_TX_PAD: R21.2
- new net VTX_RX_PAD: R7.2
- new net VTX_TX_PAD: R19.2
- no-connect marks 66 -> 59
Other:
- moved on the sheet: C17
